File: Pico.kicad_sch (KiCad schematic)
At the start: 39 parts, among them J1 DE15_Pins_HighDensity, J10 Conn_02x10_Odd_Even, J11 DB25_Socket, J2 Conn_02x10_Odd_Even, J3 Conn_02x04_Odd_Even, J5 Micro_SD_Card, J8 W5500 Lite, J9 DB25_Pins, U1 RASPBERRY_PI_PICO, U2 SN74LVC8T245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

Commit message: Fix bugs
Parts:
- removed J10: Conn_02x10_Odd_Even, Connector_PinHeader_2.54mm:PinHeader_2x10_P2.54mm_Vertical, symbol Connector_Generic:Conn_02x10_Odd_Even
- added unit 5 of U4
- added unit 3 of U4
- added unit 4 of U4
- J3: footprint Connector_PinSocket_2.54mm:PinSocket_2x04_P2.54mm_Vertical -> Connector_PinHeader_2.54mm:PinHeader_2x04_P2.54mm_Vertical
- renumbered J2 to J10
Connections:
- net +3V3: now also D1.2 (A), J11.13, J5.4 (VDD), J8.10 (Pin_10), J8.9 (Pin_9), J9.15 (P15), R15.2, U1.39 (VSYS), U2.1 (V_{CCA}), U6.36 (3V3), U4.14 (VCC); no longer U1.36 (3V3), U4.14 (VCC)
- net DRQ0: no longer U6.4 (GP2)
- net GND: now also U4.7 (GND); no longer J10.9 (Pin_9), U4.7 (GND)
- net RDYIN: no longer D6.3 (Y)
- net ~{C100}: now also D6.10 (B), D6.2 (B), J10.15 (Pin_15)
- net ~{C300}: now also D4.10 (B), D4.13 (B), D5.12 (A); no longer D4.2 (B), D4.4 (A), D5.1 (A)
- net ~{C500}: now also D4.2 (B), D4.4 (A), D5.1 (A); no longer D4.10 (B), D4.13 (B), D5.12 (A)
- net ~{I/OWR}: now also J10.9 (Pin_9)
- net ~{RD}: now also D6.1 (A); no longer U6.10 (GP7)
- net ~{WR}: now also D6.9 (A); no longer U6.9 (GP6)
- net at D9.5 (Q): no longer D6.1 (A)
- net ~{CSW3}: now reaches D6.8 (Y)
- net ~{CSW3}: now also U6.9 (GP6)
- removed net +5V: D1.2 (A), J10.15 (Pin_15), J11.13, J9.15 (P15), U1.39 (VSYS), U2.1 (V_{CCA})
- new net ~{CSR3}: D6.3 (Y), U6.10 (GP7)
- no-connect marks 22 -> 19
Other:
- moved on the sheet: D3B, D3D, D3F, D6A, D6C, U4B
