File: PicoPDC.kicad_sch (KiCad schematic)
At the start: 56 parts, among them J1 DE15_Pins_HighDensity, J10 Conn_02x10_Odd_Even, J11 DB25_Socket, J2 To PICO, J3 Conn_02x04_Odd_Even, J4 Conn_01x01_Pin, J5 Micro_SD_Card, J6 To ProgDC, J8 W5500 Lite, J9 DB25_Pins, U1 RASPBERRY_PI_PICO, U2 SN74LVC8T245, U3 74LS30, U4 74AHCT125, U5 74LS30, U6 RASPBERRY_PI_PICO, U7 74LS373, U8 74LVC1G32

Commit message: Update
Parts:
- removed D1: 1N4148WT, Diode_SMD:D_SOD-523, symbol Diode:1N4148WT
- added C3: 470, Capacitor_THT:C_Rect_L7.0mm_W2.0mm_P5.00mm, symbol Device:C
- added R22: 1K, Resistor_THT:R_Axial_DIN0207_L6.3mm_D2.5mm_P5.08mm_Vertical, symbol Device:R
- added VD5: 1N4148, Diode_THT:D_DO-34_SOD68_P2.54mm_Vertical_AnodeUp, symbol Diode:BAT43
Connections:
- net +5V: now also U6.39 (VSYS)
- net GND: now also C3.2; no longer D9.2 (D)
- net HLDA: now also R21.1; no longer R21.2
- net HOLD2: now also D3.9 (A)
- net ~{I/ORD}: no longer D3.11 (A)
- net ~{INT2}: now also R21.2; no longer R21.1
- net at D3.10 (Y): no longer D9.3 (C)
- net at U2.22 (~{OE}): now also C3.1, R22.1; no longer D5.3 (Y)
- new net: D5.3 (Y), R22.2
- no-connect marks 23 -> 31
Other:
- moved on the sheet: U4B

Commit message: Add YM2149 schematics
Parts:
- added C4, C5: 0.68, Package_SO:SOIC-8_3.9x4.9mm_P1.27mm, symbol Device:C_Small
- added C6, C7: 4.7x50V, Package_SO:SOIC-8_3.9x4.9mm_P1.27mm, symbol Device:C_Polarized
- added D12: 133LN1, Package_DIP:DIP-14_W7.62mm, symbol Pico-altium-import:root_0_133LN1_*
- added D13: 133LL1, Package_DIP:DIP-14_W7.62mm, symbol Pico-altium-import:root_0_133LL1_*
- added D8: 74HC74N, Package_DIP:DIP-14_W7.62mm_Socket, symbol VGA_Sync-altium-import:root_0_74HC74N_*
- added J12: Conn_02x13_Odd_Even, Package_CSP:Xilinx_CSG48_7.0x7.0mm_Layout7x7_P0.8mm, symbol Connector_Generic:Conn_02x13_Odd_Even
- added J13: Conn_02x08_Odd_Even, Package_CSP:Xilinx_CSG48_7.0x7.0mm_Layout7x7_P0.8mm, symbol Connector_Generic:Conn_02x08_Odd_Even
- added J14: AudioJack2_Ground, Package_LCC:PLCC-84_29.3x29.3mm_P1.27mm, symbol Connector_Audio:AudioJack2_Ground
- added J7: Conn_01x02_Pin, Package_DIP:DIP-20_W7.62mm, symbol Connector:Conn_01x02_Pin
- added R23, R24, R25, R26: 2K7, Resistor_THT:R_Axial_DIN0207_L6.3mm_D2.5mm_P5.08mm_Vertical, symbol Device:R
- added R27, R28: 1K3, Resistor_THT:R_Axial_DIN0207_L6.3mm_D2.5mm_P5.08mm_Vertical, symbol Device:R
- added U9: YM2149, Package_DIP:DIP-40_W15.24mm, symbol Audio:YM2149
- renumbered D8 to D2
Connections:
- net +3V3: now also D12.14 (VCC), D12.14 (VCC), D12.14 (VCC), D12.14 (VCC), D13.14 (VCC), D13.14 (VCC), D13.14 (VCC), D13.14 (VCC), D8.14 (VCC), D8.14 (VCC)
- net +5V: now also D8.10 (~{S}), D8.4 (~{S}), J12.2 (Pin_2), U9.25 (A8), U9.28 (BC2), U9.40 (VCC)
- net A0: no longer D11.12 (A), U3.12
- net A1: no longer D11.13 (B), U3.11
- net A10: no longer U5.6
- net A11: no longer U5.5
- net A12: no longer U5.4
- net A13: no longer U5.3
- net A14: no longer U5.2
- net A15: no longer U5.1
- net A2: no longer U3.6
- net A8: no longer U5.12
- net A9: no longer U5.11
- net D0: now also J12.3 (Pin_3), U9.37 (DA0)
- net D1: now also J12.4 (Pin_4), U9.36 (DA1)
- net D2: now also J12.5 (Pin_5), U9.35 (DA2)
- net D3: now also J12.6 (Pin_6), U9.34 (DA3)
- net D4: now also J12.7 (Pin_7), U9.33 (DA4)
- net D5: now also J12.8 (Pin_8), U9.32 (DA5)
- net D6: now also J12.9 (Pin_9), U9.31 (DA6)
- net D7: now also J12.10 (Pin_10), U9.30 (DA7)
- net GND: now also D12.7 (GND), D12.7 (GND), D12.7 (GND), D12.7 (GND), D13.7 (GND), D13.7 (GND), D13.7 (GND), D13.7 (GND), D8.7 (GND), D8.7 (GND), J12.1 (Pin_1), J14.G, R25.2, R26.1, U9.1 (VSS), U9.24 (~{A9}), U9.26 (~{SEL})
- net ~{INT2}: no longer R21.2, U6.29 (GP22)
- net ~{RESET}: now also J12.24 (Pin_24), U9.23 (~{RESET})
- net A3 renamed AB3
- net AB3: now also J13.4 (Pin_4)
- net A4 renamed AB4
- net AB4: now also J13.5 (Pin_5)
- net A5 renamed AB5
- net AB5: now also J13.6 (Pin_6)
- net A6 renamed AB6
- net AB6: now also J13.7 (Pin_7)
- net A7 renamed AB7
- net AB7: now also J13.8 (Pin_8)
- new net: R23.2, R24.1, U9.38 (C)
- new net: C5.2, C7.1, R24.2, R25.1, R28.1
- new net: D12.4 (Y), U9.27 (BDIR)
- new net: D12.6 (Y), U9.29 (BC1)
- new net: R27.2, U9.3 (A)
- new net: R28.2, U9.4 (B)
- new net: D12.3 (A), D13.11 (Y)
- new net: D13.10 (B), D13.13 (B), D13.3 (Y)
- new net: D8.12 (D), D8.5 (Q)
- new net: D12.12 (Y), D8.1 (~{R}), D8.13 (~{R}), D8.2 (D)
- new net: D13.4 (A), D8.8 (~{Q})
- new net: C4.2, C6.1, R23.1, R26.2, R27.1
- new net: C5.1, C7.2, J14.T
- new net: D12.5 (A), D13.8 (Y)
- new net: D12.11 (A), D13.6 (Y)
- new net: D12.10 (Y), D13.2 (B)
- new net: C4.1, C6.2, J14.S
- new net AB0: D11.12 (A), D13.9 (A), J12.21 (Pin_21), J13.1 (Pin_1), U3.12
- new net AB1: D11.13 (B), D13.12 (A), J12.22 (Pin_22), J13.2 (Pin_2), U3.11
- new net AB10: J13.11 (Pin_11), U5.6
- new net AB11: J13.12 (Pin_12), U5.5
- new net AB12: J13.13 (Pin_13), U5.4
- new net AB13: J13.14 (Pin_14), U5.3
- new net AB14: J13.15 (Pin_15), U5.2
- new net AB15: J13.16 (Pin_16), U5.1
- new net AB2: J13.3 (Pin_3), U3.6
- new net AB8: J13.9 (Pin_9), U5.12
- new net AB9: J13.10 (Pin_10), U5.11
- new net CLK: D13.5 (B), D8.11 (C), D8.3 (C), J7.2 (Pin_2), U9.22 (CLOCK)
- new net ~{CS_PSG}: D12.13 (A), D13.1 (A), J7.1 (Pin_1)
- new net ~{INT2}/HLDA: R21.2, U6.29 (GP22)
- no-connect marks 31 -> 34
Other:
- moved on the sheet: R19, R21

Commit message: Update PicoPDC
Other:
- note added: "OR"
- moved on the sheet: D11B, D11D, D12B, D13C, D2A, D2B, R19, U8, VD2, VD4

Commit message: Fix schemes
Connections:
- net ~{FFFF}: now reaches D10.12 (A), D10.8 (Y)
- no-connect marks 34 -> 41
Changed lines of the file:
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@@
 	)
 	(junction
+		(at -53.34 97.79)
+		(diameter 0)
+		(color 0 0 0 0)
+	)
+	(junction
 		(at 64.77 73.66)
 		(diameter 0)
@@
 	)
 	(no_connect
+		(at -173.99 134.62)
+	)
+	(no_connect
 		(at -54.61 40.64)
 	)
@@
 	)
 	(no_connect
+		(at -157.48 102.87)
+	)
+	(no_connect
 		(at -204.47 68.58)
 	)
@@
 	)
 	(no_connect
+		(at -157.48 124.46)
+	)
+	(no_connect
 		(at 54.61 63.5)
 	)
@@
 	)
 	(no_connect
+		(at 251.46 30.48)
+	)
+	(no_connect
 		(at 54.61 43.18)
 	)
@@
 	)
 	(no_connect
+		(at -173.99 121.92)
+	)
+	(no_connect
 		(at -90.17 50.8)
 	)
@@
 		(at 149.86 184.15)
 	)
+	(no_connect
+		(at -173.99 100.33)
+	)
+	(no_connect
+		(at -173.99 113.03)
+	)
 	(bus_entry
 		(at 113.03 165.1)
@@
 	(wire
 		(pts
+			(xy -53.34 97.79) (xy -52.07 97.79)
+		)
+		(stroke
+			(width 0)
+			(type default)
+		)
+	)
+	(wire
+		(pts
 			(xy -38.1 153.67) (xy -43.18 153.67)
 		)
@@
 		)
 	)
+	(wire
+		(pts
+			(xy -53.34 97.79) (xy -53.34 85.09)
+		)
+		(stroke
+			(width 0)
+			(type default)
+		)
+	)
 	(bus
 		(pts
@@
 	(wire
 		(pts
+			(xy -69.85 85.09) (xy -53.34 85.09)
+		)
+		(stroke
+			(width 0)
+			(type default)
+		)
+	)
+	(wire
+		(pts
 			(xy -73.66 143.51) (xy -68.58 143.51)
 		)
@@
 	(wire
 		(pts
-			(xy -55.88 97.79) (xy -52.07 97.79)
+			(xy -55.88 97.79) (xy -53.34 97.79)
 		)
 		(stroke
@@
 		(effects
 			(font
+				(size 1.27 1.27)
+			)
+			(justify left bottom)
+		)
+	)
+	(label "~{FFFF}"
+		(at -69.85 85.09 0)
+		(effects
+			(font
