File: stepper2/stepper2.kicad_sch (KiCad schematic)
At the start: 20 parts, among them J1 DB25_Socket, J2 Conn_02x10_Odd_Even, J3 DB25_Pins, J4 Conn_02x10_Odd_Even, J5 Blue Pill, J6 IPS 240*240, SW2 SW_Push, SW3 SW_Push, SW4 SW_SPDT, SW5 SW_Push_SPDT

Commit message: Fix schemes
Connections:
- net +5V: no longer D1.14 (VCC), D1.14 (VCC), D4.14 (VCC), J5.20 (Pin_20), J5.38 (Pin_38), J6.2 (Pin_2)
- net at D4.4 (~{S}), R4.1, SW5.1 (A): now also D1.4 (~{S}); no longer D1.1 (~{R})
- net at R3.2, SW5.3 (C): now also D1.1 (~{R}); no longer D1.4 (~{S})
- new net VCC: D1.14 (VCC), D1.14 (VCC), D4.14 (VCC), J5.20 (Pin_20), J5.38 (Pin_38), J6.2 (Pin_2)
- no-connect marks 3 -> 2
Other:
- moved on the sheet: D2, D3, J3, J4, J5, J6, R3, R4, SW2, SW3, SW5, VD2

Commit message: Fix warnings
Parts:
- D1, D4: symbol VGA_Sync-altium-import:root_0_74HC74N_* -> Retro2:root_0_74HC74N_*
- D2, D3: symbol Pico-altium-import:root_0_KR1533KP11_* -> Retro2:KR1533KP11_*
Connections:
- net 5V is gone; now on net +5V: J5.18 (Pin_18)
- net +5V: no longer D2.16 (VCC), D3.16 (VCC), R1.1, R3.1, R4.2
- net GND: no longer J5.19 (Pin_19), J5.39 (Pin_39), J5.40 (Pin_40), J6.1 (Pin_1)
- net VCC: now also D2.16 (VCC), D3.16 (VCC), R1.1, R3.1, R4.2; no longer J5.20 (Pin_20), J5.38 (Pin_38), J6.2 (Pin_2)
- net BLK: no longer names the net of J6.7 (Pin_7)
- net R renamed RESET
- net ~{I/OR} renamed ~{I/OR}
- new net +3.3V: J5.20 (Pin_20), J5.38 (Pin_38), J6.2 (Pin_2)
- new net G: J5.19 (Pin_19), J5.39 (Pin_39), J5.40 (Pin_40), J6.1 (Pin_1)
- no-connect marks 2 -> 56
Other:
- note added: "+3.3V"
- note added: "BLK"
- note added: "DC"
- note added: "GND"
- note added: "R"
- note added: "RES"
- note added: "SCK"
- note added: "SDA"
- moved on the sheet: J2

Commit message: Fix stepper
Parts:
- added unit 2 of D4
- added R5: 1K, Resistor_THT:R_Axial_DIN0207_L6.3mm_D2.5mm_P5.08mm_Vertical, symbol Device:R
- added VD3: 1N4148, Diode_THT:D_DO-34_SOD68_P2.54mm_Vertical_AnodeUp, symbol Diode:BAT43
Connections:
- net GND: now also D4.7 (GND); no longer D1.12 (D)
- net RDYIN: now also D1.9 (Q); no longer D1.8 (~{Q})
- net STB: now also SW4.3 (C); no longer SW4.1 (A)
- net VCC: now also D4.14 (VCC)
- net ~{RESET}: now also R5.1
- net at SW4.2 (B): no longer D1.10 (~{S})
- net at D4.5 (Q): now also SW4.1 (A); no longer SW4.3 (C)
- net at D4.1 (~{R}), R1.2: now also D1.10 (~{S}), D1.12 (D); no longer D1.13 (~{R})
- net at D1.4 (~{S}), R4.1, SW5.1 (A): no longer D4.4 (~{S})
- net at D1.11 (C), R2.1: now also D4.4 (~{S})
- new net: D1.13 (~{R}), R5.2
- no-connect marks 56 -> 55
Other:
- note added: "Z80 8080"
- moved on the sheet: D1B, D4A, SW4
